File: cubieboard-lora-gateway-lrwan-gs_hf1.kicad_pcb (KiCad board)
At the start: 0 parts

Commit message: Finalized project
Parts:
- added C1: 100n, Capacitors_Smd_0603:100nF_0603, F.Cu at (117.0, 115.8)
- added C2: 10uF, Capacitors_Smd_0603:10uF_10V_0603, F.Cu at (117.0, 117.3)
- added Con1: Header_Socket_2x26, Header_Socket_2mm:Header_Socket_2x26pin, B.Cu at (128.2, 73.0)
- added Con2: Header_Socket_2x26, Header_Socket_2mm:Header_Socket_2x26pin, B.Cu at (128.1, 126.0)
- added Con3: 2041119-1, Smd_Connectors:2041119-1, F.Cu at (112.9, 99.5)
- added D1: KPG-1608SURKC-T, Diodes:LED_KPG-1608SURKC-T, F.Cu at (182.3, 77.2)
- added D2: KPT-1608CGCK, Diodes:LED_KPT-1608CGCK, F.Cu at (190.2, 123.8)
- added D3: KPT-1608CGCK, Diodes:LED_KPT-1608CGCK, F.Cu at (183.5, 123.8)
- added MH1: MW_M2_Grounded, Mounting_Holes:Mounting_Hole_M2_Grounded, F.Cu at (100.7, 72.6)
- added MH2: MW_M2_Grounded, Mounting_Holes:Mounting_Hole_M2_Grounded, F.Cu at (174.3, 72.6)
- added MH3: MW_M2_Grounded, Mounting_Holes:Mounting_Hole_M2_Grounded, F.Cu at (100.7, 126.3)
- added MH4: MW_M2_Grounded, Mounting_Holes:Mounting_Hole_M2_Grounded, F.Cu at (174.3, 126.3)
- added P1: Power_Sel, Goldpin:Goldpin_3_2_54mm, F.Cu at (178.9, 83.7)
- added P2: Band_Sel1, Goldpin:Goldpin_3_2_54mm, F.Cu at (178.9, 105.4)
- added P3: Band_Sel2, Goldpin:Goldpin_3_2_54mm, F.Cu at (178.9, 117.1)
- added R1: 220R, Resistor_Smd_0603:220R_0603, F.Cu at (179.7, 77.2)
- added R2: 220R, Resistor_Smd_0603:220R_0603, F.Cu at (187.6, 123.8)
- added R3: 220R, Resistor_Smd_0603:220R_0603, F.Cu at (180.8, 123.8)
- added REF**: KiCad-Logo2_6mm_SilkScreen, Symbols:KiCad-Logo2_6mm_SilkScreen, F.Cu at (154.0, 103.8)
- added REF**: OSHW-Logo_19x20mm_SilkScreen, Symbols:OSHW-Logo_19x20mm_SilkScreen, F.Cu at (129.4, 103.2)
- added REF**: Symbol_ESD-Logo_SilkScreen, Symbols:Symbol_ESD-Logo_SilkScreen, F.Cu at (188.8, 108.3)
- added U1: LRWAN_GS_HF1, Shields:LRWAN_GS_HF1, F.Cu at (137.8, 99.5)
Routing:
- net 3V3: track 0.00 -> 169.0 mm, vias 0 -> 2
- net 5V: track 0.00 -> 128.9 mm
- net /PI10/SPI0_CS0/UART5_TX/EINT22: track 0.00 -> 80.7 mm, vias 0 -> 2
- net /PB11/I2S_D03: track 0.00 -> 77.2 mm, vias 0 -> 1
- net /PI13/SPI0_MISO/UART6_RX/EINT25: track 0.00 -> 75.6 mm, vias 0 -> 4
- net /PI12/SPI0_MOSI/UART6_TX/EINT24: track 0.00 -> 62.0 mm, vias 0 -> 2
- net /PB18/TWI1_SCK: track 0.00 -> 60.7 mm, vias 0 -> 1
- net /PI11/SPI0_CLK/UART5_RX: track 0.00 -> 59.5 mm, vias 0 -> 1
- net /PE4/TS0_D0: track 0.00 -> 58.5 mm, vias 0 -> 2
- net GND: track 0.00 -> 47.6 mm, vias 0 -> 643
- net /PE11/TS0_D7/CSI0_D7: track 0.00 -> 42.7 mm
- net Net-(P3-Pad2): track 0.00 -> 41.4 mm
- net Net-(P1-Pad2): track 0.00 -> 39.2 mm
- net Net-(P2-Pad2): track 0.00 -> 37.4 mm
- net /PE10/TS0_D6/CSI0_D6: track 0.00 -> 34.9 mm
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- added copper zone on B.Cu, net GND
- added copper zone on F.Cu, net GND
Other:
- board outline added: 100 x 60.1 mm
- copper layers 0 -> 2
- board text added: "3V3"
- board text added: "5V0"
- board text added: "BAND SELECT 1"
- board text added: "BAND SELECT 2"
- board text added: "Cubieboard Lora Gateway LRWAN-GS-HF1 RAK833"
- board text added: "POWER SELECT"
