File: cubieboard-lora-gateway-lrwan-gs_hf1.kicad_pcb (KiCad board)
At the start: 2 copper layers, 100 x 60.1 mm, 22 parts, among them Con1 Header_Socket_2x26, Con2 Header_Socket_2x26, Con3 2041119-1, P1 Power_Sel, P2 Band_Sel1, P3 Band_Sel2, U1 LRWAN_GS_HF1

Commit message: Applied issue
Routing:
- net 3V3: track 169.0 -> 170.3 mm, vias 2 -> 4
- net 5V: track 128.9 -> 129.4 mm
- net GND: vias 643 -> 641
