File: cubieboard-lora-gateway-lrwan-gs_hf1.kicad_sch (KiCad schematic)
At the start: 0 parts

Commit message: Finalized project
Parts:
- added Con1, Con2: Header_Socket_2x26, Header_Socket_2mm:Header_Socket_2x26pin, symbol Header_Socket_2mm:Header_Socket_2x26
- added D1: KPG-1608SURKC-T, Diodes:LED_KPG-1608SURKC-T, symbol Diodes:KPG-1608SURKC-T
- added D2, D3: KPT-1608CGCK, Diodes:LED_KPT-1608CGCK, symbol Diodes:KPT-1608CGCK
- added MH1, MH2, MH3, MH4: MW_M2_Grounded, Mounting_Holes:Mounting_Hole_M2_Grounded, symbol Mounting_Holes:Mounting_Hole_M2_Grounded
- added P1: Power_Sel, Goldpin:Goldpin_3_2_54mm, symbol Goldpin_2_54mm:GOLDPIN_3_2_54MM
- added P2: Band_Sel1, Goldpin:Goldpin_3_2_54mm, symbol Goldpin_2_54mm:GOLDPIN_3_2_54MM
- added P3: Band_Sel2, Goldpin:Goldpin_3_2_54mm, symbol Goldpin_2_54mm:GOLDPIN_3_2_54MM
- added R1, R2, R3: 220R, Resistor_Smd_0603:220R_0603, symbol Resistors_Smd0603:220R
- added U1: LRWAN_GS_HF1, Shields:LRWAN_GS_HF1, symbol Shields:LRWAN_GS_HF1
Connections:
- new net: D3.1 (A), R3.2
- new net: D2.1 (A), R2.2
- new net: P1.2, U1.15 (VIN)
- new net: D1.1 (A), R1.2
- new net: P2.2, U1.64 (BAND_SET1_PD15)
- new net: P3.2, U1.70 (BAND_SET2_PE9)
- new net 3V3: Con1.44, P1.1, P2.1, P3.1, R1.1
- new net 5V: Con1.43, Con2.1, P1.3
- new net CSI1_IO: Con2.3
- new net CVBS: Con2.43
- new net FMINL: Con2.21
- new net FMINR: Con2.23
- new net GND: Con1.2, Con1.20, Con1.38, Con1.42, Con1.9, Con2.19, Con2.20, Con2.25, Con2.37, D1.2 (K), D2.2 (K), D3.2 (K), MH1.1, MH2.1, MH3.1, MH4.1, P2.3, P3.3, U1.11 (GND), U1.13 (GND)
- new net HPL: Con2.45
- new net HPR: Con2.47
- new net LCD1_HSYNC: Con2.35
- new net LCD1_VSYNC: Con2.33
- new net LRADC0: Con2.41
- new net PB10/I2S_D02: Con1.40
- new net PB11/I2S_D03: Con1.39, U1.66 (RST-PF12)
- new net PB18/TWI1_SCK: Con2.6, U1.78 (GPIO2-PF15)
- new net PB19/TWI1_SDA: Con2.7
- new net PB2_PWM0: Con1.31, U1.27 (GPIO3-PF10)
- new net PD0/LCD0_D0/LVDS0_VP0: Con1.1
- new net PD10/LCD0_D10/LVDS1_VP0: Con1.14
- new net PD11/LCD0_D11/LVDS1_VN0: Con1.13
- new net PD12/LCD0_D12/LVDS1_VP1: Con1.16
- new net PD13/LCD0_D13/LVDS1_VN1: Con1.15
- new net PD14/LCD0_D14/LVDS1_VP2: Con1.18
- new net PD14/LCD0_D15/LVDS1_VN2: Con1.17
- new net PD16/LCD0_D16/LVDS1_VPC: Con1.19
- new net PD17/LCD0_D17/LVDS1_VNC: Con1.22
- new net PD18/LCD0_D18/LVDS1_VP3: Con1.21
- new net PD19/LCD0_D19/LVDS1_VN3: Con1.24
- new net PD1/LCD0_D1/LVDS0_VN0: Con1.4
- new net PD20/LCD0_D20/CSI1_MCLK: Con1.23
- new net PD21/LCD0_D21/SMC_VPPEN: Con1.26
- new net PD22/LCD0_D22/SMC_VPPPP: Con1.25
- new net PD23/LCD0_D23/SMC_DET: Con1.28
- new net PD24/LCD0_CLK/SMC_VCCEN: Con1.29
- new net PD25/LCD0_DE/SMC_RST: Con1.32
- new net PD26/LCD0_HSYNC/SMC_SCK: Con1.30
- new net PD27/LCD0_VSYNC/SMC_SDA: Con1.27
- new net PD2/LCD0_D2/LVDS0_VP1: Con1.3
- new net PD3/LCD0_D3/LVDS0_VN1: Con1.6
- new net PD4/LCD0_D4/LVDS0_VP2: Con1.5
- new net PD5/LCD0_D5/LVDS0_VN2: Con1.8
- new net PD6/LCD0_D6/LVDS0_VPC: Con1.7
- new net PD7/LCD0_D7/LVDS0_VNC: Con1.10
- new net PD8/LCD0_D8/LVDS0_VP3: Con1.12
- new net PD9/LCD0_D0/LVDS0_VN3: Con1.11
- new net PE10/TS0_D6/CSI0_D6: Con2.46, R3.1
- new net PE11/TS0_D7/CSI0_D7: Con2.48, R2.1
- new net PE4/TS0_D0: Con2.34, U1.25 (GPIO4-PF5)
- new net PE5/TS0_D1/CSI0_D1/SMC_VPPEN: Con2.36, U1.74 (GPIO1-PF14)
- new net PE6/TS0_D2/CSI0_D2: Con2.38, U1.68 (GPIO0-PF13)
- new net PE7/TS0_D3/CSI0_D3: Con2.40
- new net PE8/TS0_D4/CSI0_D4: Con2.42
- new net PE9/TS0_D5/CSI0_D5: Con2.44
- new net PG0/TS1_CLK/CSI1_PCK/SDC1_CMD: Con2.5
- new net PG10/TS1_D6/CSI1_D6/UART4_TX/CSI0_D14: Con2.17
- new net PG10/TS1_D7/CSI1_D7/UART4_RX/CSI0_D15: Con2.18
- new net PG1/TS1_ERR/CSI1_CK/SDC1_CLK: Con2.10
- new net PG2/TS1_SYNC/CSI1_HSYNC/SDC1_D0: Con2.9
- new net PG3/TS1_DVLD/CSI1_VSYNC/SDC1_D1: Con2.8
- new net PG4/TS1_D0/CSI1_D0/SDC1_D2/CSI0_D8: Con2.11
- new net PG5/TS1_D1/CSI1_D1/SDC1_D3/CSI0_D9: Con2.12
- new net PG6/TS1_D2/CSI1_D2/UART3_TX/CSI0_D10: Con2.13
- new net PG7/TS1_D3/CSI1_D3/UART3_RX/CSI0_D11: Con2.14
- new net PG8/TS1_D4/CSI1_D4/UART3_RTS/CSI0_D12: Con2.15
- new net PG9/TS1_D5/CSI1_D5/UART3_CTS/CSI0_D13: Con2.16
- new net PH14/LCD1_D14/ATA_D10/KP_INT4/SMC_VPPEN/EINT14/CSI1_D14: Con2.4
- new net PH15/LCD1_D15/ATA_D11/KP_IN5/SMC_VPPPP/EINT15/CSI1_D15: Con2.2
- new net PH7/LCD1_D07/ATA_D03/UART5_RX/MS_CLK/EINT7: Con1.37
- new net PI10/SPI0_CS0/UART5_TX/EINT22: Con1.45, U1.72 (CSN-PE11)
- new net PI11/SPI0_CLK/UART5_RX: Con1.47, U1.92 (SCK-PE12)
- new net PI12/SPI0_MOSI/UART6_TX/EINT24: Con1.46, U1.94 (MOSI-PE14)
- new net PI13/SPI0_MISO/UART6_RX/EINT25: Con1.48, U1.76 (MISO-PE13)
- new net PI4_SDC3_CMD: Con2.22
- new net PI5/SDC3_CLK: Con2.24
- new net PI6/SDC3_D0: Con2.26
- new net PI7/SDC3_D1: Con2.28
- new net PI8/SDC3_D2: Con2.30
- new net PI9/SDC3_D3: Con2.32
- new net SPDIF: Con1.41
- new net VCC-RTC: Con2.39
- new net VGA_B: Con2.31
- new net VGA_G: Con2.29
- new net VGA_R: Con2.27
- new net XN_TP: Con1.36
- new net XP_TP: Con1.34
- new net YN_TP: Con1.35
- new net YP_TP: Con1.33
- no-connect marks 0 -> 6
Other:
- added sheet Minipci Module (minipci_module.kicad_sch)
- note added: "Connected"
- note added: "Heartbeat"
- note added: "Power"
- company: (none) -> MWLinux
- title: (none) -> Cubieboard 1 carrier board with lora gateway - lrwan gs hf1
